Commit message: with localization working

File: my_robot/description/gazebo_control.xacro (robot description, xacro)
@@ -16,5 +16,5 @@
             <publish_odom>true</publish_odom>
             <publish_odom_tf>true</publish_odom_tf>
-            <publish_wheel_tf>true</publish_wheel_tf>
+            <publish_wheel_tf>false</publish_wheel_tf>
         </plugin>
     </gazebo>

File: my_robot/description/robot_core.xacro (robot description, xacro)
@@ -157,4 +157,6 @@
     <gazebo reference="left_back_wheel">
         <material>Gazebo/Blue</material>
+        <mu1>0.001</mu1>
+        <mu2>0.001</mu2>
     </gazebo>
     <!-- RIGHT back WHEEL LINK -->
@@ -162,5 +164,5 @@
         <parent link="base_link"/>
         <child link="right_back_wheel"/>
-        <origin xyz="0.012 -0.175 0" rpy="${pi/2} 0 0" />
+        <origin xyz="0.0 -0.175 0" rpy="${pi/2} 0 0" />
         <axis xyz="0 0 -1"/>
     </joint>
@@ -183,4 +185,6 @@
     <gazebo reference="right_back_wheel">
         <material>Gazebo/Blue</material>
+        <mu1>0.001</mu1>
+        <mu2>0.001</mu2>
     </gazebo>
 </robot>
